File: 1. PCB/v1.0/board.brd (EAGLE design)
At the start: 69.5 x 114 mm, 2 parts

Commit message: no message
Parts:
- added U$1: GBP_POWER_JACK, ,giltesa:GBP_POWER_JACK
- added X1: (no value), ,giltesa:USB-C_6P
Connections:
- new net VCC: U$1.VCC
Other:
- board size 69.5 x 114 mm -> 69.5 x 131.9 mm

Commit message: no message
Parts:
- removed X1: (no value), ,giltesa:USB-C_6P
- U$1: value GBP_POWER_JACK -> (none)
- moved U$1 18.0 mm to (40.8, 0.16), flipped to the bottom
- moved E$2 2.24 mm to (0.48, -2.05)
Other:
- board size 69.5 x 131.9 mm -> 69.5 x 114 mm
Changed lines of the file:
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@@
 <setting verticaltext="up"/>
 </settings>
-<grid distance="5" unitdist="mil" unit="mil" style="lines" multiple="1" display="yes" altdistance="0.025" altunitdist="inch" altunit="inch"/>
+<grid distance="5" unitdist="mil" unit="mm" style="lines" multiple="1" display="yes" altdistance="0.025" altunitdist="inch" altunit="inch"/>
 <layers>
 <layer number="1" name="Top" color="4" fill="1" visible="yes" active="yes"/>
@@
 <layer number="21" name="tPlace" color="7" fill="1" visible="yes" active="yes"/>
 <layer number="22" name="bPlace" color="7" fill="1" visible="yes" active="yes"/>
-<layer number="23" name="tOrigins" color="15" fill="1" visible="no" active="yes"/>
-<layer number="24" name="bOrigins" color="15" fill="1" visible="no" active="yes"/>
+<layer number="23" name="tOrigins" color="15" fill="1" visible="yes" active="yes"/>
+<layer number="24" name="bOrigins" color="15" fill="1" visible="yes" active="yes"/>
 <layer number="25" name="tNames" color="7" fill="1" visible="yes" active="yes"/>
 <layer number="26" name="bNames" color="7" fill="1" visible="yes" active="yes"/>
@@
 <rectangle x1="-0.05" y1="113.75185" x2="69.49" y2="113.85176875" layer="46"/>
 <rectangle x1="-0.05" y1="113.85176875" x2="69.49" y2="113.95168125" layer="46"/>
-<hole x="37.846" y="6.477" drill="3"/>
-<hole x="40.767" y="8.763" drill="3"/>
-<hole x="43.815" y="7.493" drill="3"/>
-<hole x="38.227" y="2.032" drill="3"/>
-<hole x="43.307" y="2.032" drill="3"/>
-<hole x="46.863" y="11.43" drill="1"/>
-<wire x1="36.068" y1="0.127" x2="40.767" y2="0.127" width="0.4064" layer="21"/>
-<wire x1="40.767" y1="0.127" x2="48.006" y2="0.127" width="0.4064" layer="21"/>
-<wire x1="48.006" y1="0.127" x2="48.006" y2="12.446" width="0.4064" layer="21"/>
-<wire x1="48.006" y1="12.446" x2="46.228" y2="12.446" width="0.4064" layer="21"/>
-<wire x1="46.228" y1="12.446" x2="44.958" y2="11.176" width="0.4064" layer="21"/>
-<wire x1="44.958" y1="11.176" x2="40.767" y2="11.176" width="0.4064" layer="21"/>
-<wire x1="40.767" y1="11.176" x2="36.068" y2="11.176" width="0.4064" layer="21"/>
-<wire x1="36.068" y1="11.176" x2="36.068" y2="0.127" width="0.4064" layer="21"/>
-<hole x="46.99" y="3.81" drill="1"/>
-<wire x1="36.068" y1="-1.873" x2="48.006" y2="-1.873" width="0.4064" layer="21"/>
-<wire x1="40.767" y1="11.176" x2="40.767" y2="0.127" width="0.4064" layer="21"/>
-<wire x1="33.528" y1="-6.604" x2="33.528" y2="-16.637" width="0.4064" layer="20"/>
-<wire x1="33.528" y1="-16.637" x2="34.798" y2="-17.907" width="0.4064" layer="20" curve="90"/>
-<wire x1="34.798" y1="-17.907" x2="45.212" y2="-17.907" width="0.4064" layer="20"/>
-<wire x1="45.212" y1="-17.907" x2="46.482" y2="-16.637" width="0.4064" layer="20" curve="90"/>
-<wire x1="46.482" y1="-16.637" x2="46.482" y2="-7.62" width="0.4064" layer="20"/>
-<wire x1="46.482" y1="-7.62" x2="45.212" y2="-6.35" width="0.4064" layer="20" curve="90"/>
-<wire x1="45.212" y1="-6.35" x2="36.449" y2="-6.35" width="0.4064" layer="20"/>
-<wire x1="36.449" y1="-6.35" x2="35.941" y2="-5.842" width="0.4064" layer="20"/>
-<wire x1="35.941" y1="-5.842" x2="34.29" y2="-5.842" width="0.4064" layer="20"/>
-<wire x1="34.29" y1="-5.842" x2="33.528" y2="-6.604" width="0.4064" layer="20" curve="90"/>
-<hole x="40.767" y="-13.46" drill="1"/>
-<hole x="40.767" y="-17.873" drill="1"/>
+<wire x1="36.5" y1="0" x2="52.5" y2="0" width="0.4064" layer="21"/>
+<wire x1="47" y1="4.5" x2="47" y2="11" width="0.4064" layer="21"/>
+<wire x1="47" y1="11" x2="47" y2="11.5" width="0.4064" layer="21"/>
+<wire x1="47" y1="11.5" x2="47" y2="19.5" width="0.4064" layer="21"/>
+<wire x1="47" y1="19.5" x2="36.5" y2="19.5" width="0.4064" layer="21"/>
+<wire x1="36.5" y1="19.5" x2="36.5" y2="12" width="0.4064" layer="21"/>
+<wire x1="36.5" y1="12" x2="36.5" y2="0" width="0.4064" layer="21"/>
+<wire x1="47" y1="11.5" x2="46.5" y2="11.5" width="0.4064" layer="21"/>
+<wire x1="46.5" y1="11.5" x2="46.5" y2="11" width="0.4064" layer="21"/>
+<wire x1="46.5" y1="11" x2="47" y2="11" width="0.4064" layer="21"/>
+<wire x1="36.5" y1="12" x2="26.5" y2="12" width="0.4064" layer="21"/>
+<wire x1="26.5" y1="12" x2="26.5" y2="19.5" width="0.4064" layer="21"/>
+<wire x1="26.5" y1="19.5" x2="36.5" y2="19.5" width="0.4064" layer="21"/>
+<wire x1="21.5" y1="14.5" x2="73" y2="14.5" width="0.4064" layer="90"/>
+<circle x="22.733" y="22.352" radius="2.25" width="0.127" layer="22"/>
+<circle x="46.736" y="22.352" radius="2.25" width="0.127" layer="22"/>
+<wire x1="34.75" y1="-4.5" x2="34.75" y2="25.5" width="0.4064" layer="90"/>
+<wire x1="26.95" y1="-4.5" x2="26.95" y2="25.5" width="0.4064" layer="90"/>
+<wire x1="42.55" y1="-4.5" x2="42.55" y2="25.5" width="0.4064" layer="90"/>
+<wire x1="21.5" y1="10" x2="73" y2="10" width="0.4064" layer="90"/>
+<hole x="67.54" y="11" drill="0.6"/>
+<wire x1="57.5" y1="10.5" x2="65.5" y2="10.5" width="0.4064" layer="51"/>
+<wire x1="65.5" y1="10.5" x2="66.5" y2="9.5" width="0.4064" layer="51"/>
+<wire x1="66.5" y1="9.5" x2="68" y2="9.5" width="0.4064" layer="51"/>
+<wire x1="68" y1="9.5" x2="68" y2="14" width="0.4064" layer="51"/>
+<wire x1="68" y1="14" x2="66.5" y2="14" width="0.4064" layer="51"/>
+<wire x1="66.5" y1="14" x2="65.5" y2="13" width="0.4064" layer="51"/>
+<wire x1="65.5" y1="13" x2="56" y2="13" width="0.4064" layer="51"/>
+<wire x1="51.5" y1="8.5" x2="51.5" y2="4.5" width="0.4064" layer="51"/>
+<wire x1="52.5" y1="0" x2="54" y2="0" width="0.4064" layer="51"/>
+<wire x1="54" y1="0" x2="54" y2="7" width="0.4064" layer="51"/>
+<wire x1="54" y1="7" x2="57.5" y2="10.5" width="0.4064" layer="51"/>
+<wire x1="51.5" y1="4.5" x2="47" y2="4.5" width="0.4064" layer="51"/>
+<wire x1="51.5" y1="8.5" x2="56" y2="13" width="0.4064" layer="51"/>
+<wire x1="53.54" y1="-4.5" x2="53.54" y2="25.5" width="0.4064" layer="90"/>
+<wire x1="40.767" y1="1" x2="40.767" y2="-1" width="0.4064" layer="51"/>
+<hole x="44.934" y="17.223" drill="0.6"/>
+<hole x="49.633" y="6.301" drill="0.6"/>
 </plain>
 <attributes>
@@
 <elements>
 <element name="E$1" library="CAD Ruler_EagleCad Gridrunner XL Metric V1 (Rupert Hirst 2011)" package="RULER" value="" x="-0.0508" y="114.9952"/>
-<element name="E$2" library="CAD Ruler_EagleCad Gridrunner XL Metric V1 (Rupert Hirst 2011)" package="RULER" value="" x="-0.5182" y="-0.0508" rot="R90"/>
-<element name="U$1" library=",giltesa" package="GBP_POWER_JACK" value="GBP_POWER_JACK" x="40.767" y="-17.873"/>
-<element name="X1" library=",giltesa" package="USB-C_6P" value="" x="40.767" y="-13.46"/>
+<element name="E$2" library="CAD Ruler_EagleCad Gridrunner XL Metric V1 (Rupert Hirst 2011)" package="RULER" value="" x="0.4818" y="-2.0508" rot="R90"/>
+<element name="U$1" library=",giltesa" package="GBP_POWER_JACK" value="" x="40.767" y="0.161" rot="MR0"/>
 </elements>
 <signals>
