File: 1. PCB/v1.0/board.sch (EAGLE design)
At the start: 2 parts

Commit message: no message
Parts:
- removed X1: (no value), ,giltesa:USB-CPOWER
- U$1: value GBP_POWER_JACK -> (none)
Changed lines of the file:
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@@
 <parts>
 <part name="U$1" library=",giltesa" deviceset="GBP_POWER_JACK" device=""/>
-<part name="X1" library=",giltesa" deviceset="USB-C" device="POWER"/>
 </parts>
 <sheets>
@@
 <instances>
 <instance part="U$1" gate="G$1" x="10.16" y="17.78"/>
-<instance part="X1" gate="G$1" x="12.7" y="45.72"/>
 </instances>
 <busses>
